Commit message: added offsets, gripper mass change much effect

File: ros2_ws/src/manipulators/assets/robots/kinova/urdf/gen3_2f85.urdf (robot description, URDF)
Before this commit: robot gen3_, 21 links, 20 joints
Links:
- link wrist_camera_mount_link: mass 0.4 -> 0.5

Commit message: latest

File: ros2_ws/src/manipulators/assets/robots/kinova/urdf/gen3_2f85.urdf (robot description, URDF)
Before this commit: robot gen3_, 21 links, 20 joints
Links:
- link gen3_robotiq_85_base_link: mass 5.14e-01 -> 0.514
